File: topboard/topboard.sch (EAGLE design)
At the start: 53 parts, among them U3 XBEE-1B2

Commit message: topboard fixed during worksession
Change-Id: Ie840baea4df49c21f43eef8b219610f24d1802e3
Parts:
- removed GAME: Game, pinhead-2:PINHD-1X04_2.54-S
- removed U$1: PANDAPWR, Custom:PANDAPWR
- added 0, 1, 2, 3, 4, 5: (no value), pinhead-2:PINHD-1X04_2.54-S
- added ACCELEROMETER: MMA8451QT, MMA8451QT:MMA8451QT
- added C5, C6: 0.1u, SparkFun:CAP0603-CAP
- added C7: 4.7u, SparkFun:CAP0603-CAP
- added JP3: (no value), SparkFun:M02PTH4
- added R10, R9: 4.7k, SparkFun:RESISTOR0603-RES
- added RFID: (no value), pinhead:PINHD-1X6
- added SOLENOID: (no value), pinhead:PINHD-1X4
- C3, C4: value (none) -> .1uF
- IR: value GYRO -> (none)
- LED1, LED2, LED3, LED4: device led:LED5MM -> SparkFun:LED0603
- R4, R5, R6: value (none) -> 200
- R8: value (none) -> 220K
- SERVO: value Servos -> (none)
- renumbered GYRO to IR
Connections:
- new net IO59/INT@2: ACCELEROMETER.INT@2
- new net IO60/INT@1: ACCELEROMETER.INT@1
- new net N$10: ACCELEROMETER.BYP, C6.1
- new net N$9: ACCELEROMETER.GND@3, C7.2
- net 12V: now also JP3.2; no longer U$1.12V
- net GND: now also 0.1, 1.1, 2.1, 3.1, 4.1, 5.1, ACCELEROMETER.GND@2, ACCELEROMETER.SA0, C5.2, C6.2, JP3.1, RFID.1; no longer GAME.1, U$1.GND
- net IO10/SCK1: now also RFID.3
- net IO6/MOSI1: now also RFID.5
- net IO61: now also SOLENOID.3
- net IO64: now also SOLENOID.2
- net IO66: now also SOLENOID.1
- net IO67: now also RFID.6
- net IO68: now also SOLENOID.4
- net IO8/MISO1: now also RFID.4
- net SCL0/IO31*: now also 0.4, 1.4, 2.4, 3.4, 4.4, 5.4, ACCELEROMETER.SCL, R9.1; no longer GAME.4
- net SDA0/IO33*: now also 0.3, 1.3, 2.3, 3.3, 4.3, 5.3, ACCELEROMETER.SDA, R10.1; no longer GAME.3
- net VCC: now also 0.2, 1.2, 2.2, 3.2, 4.2, 5.2, ACCELEROMETER.VDD, ACCELEROMETER.VVDIO, C5.1, C7.1, R10.2, R9.2, RFID.2; no longer GAME.2
Other:
- note added: "Game Sensors"
- note added: "Solenoid"
