File: simple_ext/SimpleExt.brd (EAGLE design)
At the start: 45.4 x 30.1 mm, 23 parts, among them IC2 74ALS08D

Commit message: added copyright stuff and open source logo
Change-Id: Ia149b3f1e75c81f992df6b9b6b68b519a3d9cc7f
Parts:
- removed U$4: (no value), pie:PIE-LOGO-SMALL
- added U$2: (no value), pie:OSHW-LOGO-S
Other:
- board text added: "Copyright (c) 2013, Pioneers in Engineering All rights reserved. Design by: Jared Porter This design is open source hardware. For more information, visit pioneers.berkeley.edu/opensource"
Changed lines of the file:
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@@
 <?xml version="1.0" encoding="utf-8"?>
 <!DOCTYPE eagle SYSTEM "eagle.dtd">
-<eagle version="6.1">
+<eagle version="6.3">
 <drawing>
 <settings>
@@
 <layer number="20" name="Dimension" color="15" fill="1" visible="yes" active="yes"/>
 <layer number="21" name="tPlace" color="7" fill="1" visible="yes" active="yes"/>
-<layer number="22" name="bPlace" color="7" fill="1" visible="yes" active="yes"/>
+<layer number="22" name="bPlace" color="14" fill="1" visible="yes" active="yes"/>
 <layer number="23" name="tOrigins" color="15" fill="1" visible="yes" active="yes"/>
 <layer number="24" name="bOrigins" color="15" fill="1" visible="yes" active="yes"/>
@@
 <layer number="106" name="bPlate" color="7" fill="1" visible="yes" active="yes"/>
 <layer number="107" name="Crop" color="7" fill="1" visible="yes" active="yes"/>
+<layer number="108" name="fp8" color="7" fill="1" visible="yes" active="yes"/>
+<layer number="109" name="fp9" color="7" fill="1" visible="yes" active="yes"/>
+<layer number="110" name="fp0" color="7" fill="1" visible="yes" active="yes"/>
 <layer number="116" name="Patch_BOT" color="9" fill="4" visible="yes" active="yes"/>
 <layer number="121" name="_tsilk" color="7" fill="1" visible="yes" active="yes"/>
 <layer number="122" name="_bsilk" color="7" fill="1" visible="yes" active="yes"/>
+<layer number="123" name="tTestmark" color="7" fill="1" visible="yes" active="yes"/>
+<layer number="124" name="bTestmark" color="7" fill="1" visible="yes" active="yes"/>
+<layer number="125" name="_tNames" color="7" fill="1" visible="yes" active="yes"/>
+<layer number="131" name="tAdjust" color="7" fill="1" visible="yes" active="yes"/>
+<layer number="132" name="bAdjust" color="7" fill="1" visible="yes" active="yes"/>
+<layer number="144" name="Drill_legend" color="7" fill="1" visible="yes" active="yes"/>
 <layer number="151" name="HeatSink" color="7" fill="1" visible="yes" active="yes"/>
 <layer number="199" name="Contour" color="7" fill="1" visible="no" active="no"/>
@@
 <layer number="213" name="213bmp" color="7" fill="1" visible="yes" active="yes"/>
 <layer number="214" name="214bmp" color="7" fill="1" visible="yes" active="yes"/>
+<layer number="215" name="215bmp" color="7" fill="1" visible="yes" active="yes"/>
+<layer number="216" name="216bmp" color="7" fill="1" visible="yes" active="yes"/>
+<layer number="217" name="217bmp" color="18" fill="1" visible="no" active="no"/>
+<layer number="218" name="218bmp" color="19" fill="1" visible="no" active="no"/>
+<layer number="219" name="219bmp" color="20" fill="1" visible="no" active="no"/>
+<layer number="220" name="220bmp" color="21" fill="1" visible="no" active="no"/>
+<layer number="221" name="221bmp" color="22" fill="1" visible="no" active="no"/>
+<layer number="222" name="222bmp" color="23" fill="1" visible="no" active="no"/>
+<layer number="223" name="223bmp" color="24" fill="1" visible="no" active="no"/>
+<layer number="224" name="224bmp" color="25" fill="1" visible="no" active="no"/>
 <layer number="250" name="Descript" color="3" fill="1" visible="no" active="no"/>
 <layer number="251" name="SMDround" color="12" fill="11" visible="no" active="no"/>
@@
 <text x="17.78" y="30.48" size="0.8128" layer="22" font="vector" rot="MR0">Pioneers in Engineering</text>
 <text x="17.78" y="29.21" size="0.8128" layer="22" font="vector" rot="MR0">Simple Extension 2/3/12</text>
+<text x="16.51" y="2.54" size="0.3048" layer="22" font="vector" rot="MR0">Copyright (c) 2013, Pioneers in Engineering
+All rights reserved.
+Design by: Jared Porter
+This design is open source hardware.
+For more information, visit pioneers.berkeley.edu/opensource</text>
 </plain>
 <attributes>
@@
 </class>
 </classes>
-<designrules>
+<designrules name="default">
 <description language="de">&lt;b&gt;EAGLE Design Rules&lt;/b&gt;
 &lt;p&gt;
@@
 <element name="C1" library="rcl" package="C0603K" value="" x="33.02" y="11.43" rot="R270"/>
 <element name="JP2" library="pinhead" package="2X03" value="" x="40.259" y="8.001" rot="R270"/>
-<element name="U$4" library="pie" package="PIE-LOGO-SMALL" value="" x="12.7" y="7.62" rot="MR0"/>
 <element name="U$5" library="pie" package="PIE-LOGO-SMALL" value="" x="12.7" y="16.51" rot="MR0"/>
 <element name="U$6" library="pie" package="PIE-LOGO-SMALL" value="" x="12.7" y="25.4" rot="MR0"/>
+<element name="U$2" library="pie" package="OSHW-LOGO-S" value="" x="2.54" y="6.35" rot="MR0"/>
 </elements>
 <signals>
@@
 </board>
 </drawing>
+<compatibility>
+<note version="6.3" minversion="6.2.2" severity="warning">
+Since Version 6.2.2 text objects can contain more than one line,
+which will not be processed correctly with this version.
+</note>
+</compatibility>
 </eagle>
