File: grizzly_bear/grizzly_bear_revF.sch (EAGLE design)
At the start: 60 parts, among them Q1 N-CHANNEL-MOSFET, Q2 N-CHANNEL-MOSFET, Q3 N-CHANNEL-MOSFET, Q4 N-CHANNEL-MOSFET, Q5 IPD90P03P4L, U1 A4940, U2 ATMEGA32U4-AU, U3 ACS714, U4 UA78L00, Y1 16MHz

Commit message: Grizzly Revision B 11/10/13
Parts:
- removed STANDOFF3: STAND-OFF, pie:STAND-OFF
Changed lines of the file:
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@@
 <part name="U$19" library="pie" deviceset="XT60CONNECTOR" device=""/>
 <part name="STANDOFF4" library="pie" deviceset="STAND-OFF" device=""/>
-<part name="STANDOFF3" library="pie" deviceset="STAND-OFF" device=""/>
 <part name="FRAME1" library="pie" deviceset="FRAME-LETTER" device="">
 <attribute name="AUTHOR" value="Keegan Mann, Jay Chenn, Robert Ou"/>
@@
 <instance part="U$19" gate="G$1" x="137.16" y="45.72" rot="R270"/>
 <instance part="STANDOFF4" gate="G$1" x="144.78" y="2.54" rot="R90"/>
-<instance part="STANDOFF3" gate="G$1" x="144.78" y="7.62" rot="R90"/>
 <instance part="FRAME1" gate="G$1" x="0" y="0"/>
 <instance part="FRAME1" gate="G$2" x="147.32" y="0">
