File: eda/metal_detector_circuit.brd (EAGLE design)
At the start: 33 x 27.9 mm, 12 parts, among them IC1 555TIMER

Commit message: fixed rev label
Other:
- board text added: "v1 revA 05 Nov 2015"
- board text removed: "v1 revA 11 Nov 2015"
Changed lines of the file:
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@@
 <grid distance="0.1" unitdist="inch" unit="inch" style="lines" multiple="1" display="yes" altdistance="0.005" altunitdist="inch" altunit="inch"/>
 <layers>
-<layer number="1" name="Top" color="4" fill="1" visible="no" active="yes"/>
+<layer number="1" name="Top" color="4" fill="1" visible="yes" active="yes"/>
 <layer number="2" name="Route2" color="1" fill="3" visible="no" active="no"/>
 <layer number="3" name="Route3" color="20" fill="3" visible="no" active="no"/>
@@
 <layer number="19" name="Unrouted" color="14" fill="1" visible="yes" active="yes"/>
 <layer number="20" name="Dimension" color="15" fill="1" visible="yes" active="yes"/>
-<layer number="21" name="tPlace" color="16" fill="1" visible="no" active="yes"/>
+<layer number="21" name="tPlace" color="16" fill="1" visible="yes" active="yes"/>
 <layer number="22" name="bPlace" color="17" fill="1" visible="yes" active="yes"/>
-<layer number="23" name="tOrigins" color="15" fill="1" visible="no" active="yes"/>
+<layer number="23" name="tOrigins" color="15" fill="1" visible="yes" active="yes"/>
 <layer number="24" name="bOrigins" color="15" fill="1" visible="yes" active="yes"/>
-<layer number="25" name="tNames" color="18" fill="1" visible="no" active="yes"/>
+<layer number="25" name="tNames" color="18" fill="1" visible="yes" active="yes"/>
 <layer number="26" name="bNames" color="19" fill="1" visible="yes" active="yes"/>
-<layer number="27" name="tValues" color="18" fill="1" visible="no" active="yes"/>
+<layer number="27" name="tValues" color="18" fill="1" visible="yes" active="yes"/>
 <layer number="28" name="bValues" color="19" fill="1" visible="yes" active="yes"/>
 <layer number="29" name="tStop" color="7" fill="3" visible="yes" active="yes"/>
@@
 <wire x1="33.02" y1="27.94" x2="0" y2="27.94" width="0.254" layer="20"/>
 <wire x1="0" y1="27.94" x2="0" y2="0" width="0.254" layer="20"/>
-<text x="32.2072" y="23.1902" size="0.9144" layer="16" font="vector" ratio="20" rot="MR0">v1 revA
-11 Nov 2015</text>
+<text x="3.0988" y="6.8072" size="0.9144" layer="1" font="vector" ratio="20" rot="R90">v1 revA
+05 Nov 2015</text>
 <text x="26.67" y="26.416" size="0.762" layer="22" font="vector" ratio="20" rot="MR270">(c) Pioneers in Engineering.
 Design by:  Jaron Armiger
@@
 <wire x1="30.861" y1="17.272" x2="30.861" y2="15.24" width="0.4064" layer="1"/>
 </signal>
-<signal name="S$1">
-<wire x1="23.876" y1="20.066" x2="24.511" y2="20.066" width="0" layer="19" extent="1-16"/>
-</signal>
 <signal name="S$3">
